File: ESP-HI-PLUS.kicad_pcb (KiCad board)
At the start: 4 copper layers, 56.5 x 34 mm, 80 parts, among them J1 0.71" LCD, J2 USB_C_Receptacle_USB2.0_14P, J4 PR5L4015-5P-C-F, J5 PR5L4015-5P-C-F, Q1 NTK3139P, Q2 AO3401A, SW1 MST-12D18G5, SW2 SKRPACE010, SW3 SKRPACE010, U1 ESP32-S3-WROOM-1, U2 DMM-4026-B-I2S-R, U3 MAX98357A, U4 LSM6DSV16X, U5 MAX40200AUK, U6 TLV75733PDBV, U7 TP4065, U8 MAX40200AUK

Commit message: layout completed
Parts:
- removed the R15 at (33.8, 64.1)
- removed the R16 at (33.8, 66.8)
- added C19: 4n7, Capacitor_SMD:C_0402_1005Metric, F.Cu at (119.0, 60.5)
- added C7: 0u1, Capacitor_SMD:C_0402_1005Metric, F.Cu at (135.0, 48.0)
- added R27: 1M, PCM_Resistor_SMD_AKL:R_0402_1005Metric, F.Cu at (118.0, 60.5)
- C1: renamed from C6; footprint Capacitor_SMD:C_0603_1608Metric -> Capacitor_SMD:C_0402_1005Metric
- C10: renamed from C5; footprint Capacitor_SMD:C_0603_1608Metric -> Capacitor_SMD:C_0402_1005Metric
- C11: renamed from C16; footprint Capacitor_SMD:C_0603_1608Metric -> Capacitor_SMD:C_0402_1005Metric
- C12: renamed from C15; footprint Capacitor_SMD:C_1210_3225Metric -> Capacitor_SMD:C_0402_1005Metric
- C13: renamed from C8; footprint Capacitor_SMD:C_0603_1608Metric -> Capacitor_SMD:C_0402_1005Metric
- C14: renamed from C9; footprint Capacitor_SMD:C_0603_1608Metric -> Capacitor_SMD:C_0402_1005Metric
- C15: renamed from C11; footprint Capacitor_SMD:C_0603_1608Metric -> Capacitor_SMD:C_0402_1005Metric
- C16: renamed from C13; footprint Capacitor_SMD:C_0603_1608Metric -> Capacitor_SMD:C_0402_1005Metric
- C17: renamed from C12; footprint Capacitor_SMD:C_0603_1608Metric -> Capacitor_SMD:C_0402_1005Metric
- C18: renamed from C14; footprint Capacitor_SMD:C_0603_1608Metric -> Capacitor_SMD:C_0402_1005Metric
- C2: renamed from C7; footprint Capacitor_SMD:C_0603_1608Metric -> Capacitor_SMD:C_0402_1005Metric
- C3: renamed from C2; footprint Capacitor_SMD:C_0603_1608Metric -> Capacitor_SMD:C_0402_1005Metric
- C4: renamed from C1; footprint Capacitor_SMD:C_0603_1608Metric -> Capacitor_SMD:C_0402_1005Metric
- C5: renamed from C4; footprint Capacitor_SMD:C_0603_1608Metric -> Capacitor_SMD:C_0402_1005Metric
- C6: renamed from C3; footprint Capacitor_SMD:C_0603_1608Metric -> Capacitor_SMD:C_0402_1005Metric
- C8: renamed from C17; footprint Capacitor_SMD:C_0603_1608Metric -> Capacitor_SMD:C_0402_1005Metric
- C9: renamed from C10; footprint Capacitor_SMD:C_0603_1608Metric -> Capacitor_SMD:C_0402_1005Metric
- D6: value P4SMA6.8CA -> TGL34-6.8CA; footprint PCM_Diode_SMD_AKL:D_SMA_TVS -> PCM_Diode_SMD_AKL:D_MiniMELF_TVS
- R1: renamed from R7; footprint PCM_Resistor_SMD_AKL:R_0603_1608Metric -> PCM_Resistor_SMD_AKL:R_0402_1005Metric
- R10: renamed from R17; footprint PCM_Resistor_SMD_AKL:R_0603_1608Metric -> PCM_Resistor_SMD_AKL:R_0402_1005Metric
- R11: renamed from R18; footprint PCM_Resistor_SMD_AKL:R_0603_1608Metric -> PCM_Resistor_SMD_AKL:R_0402_1005Metric
- R12: renamed from R3; footprint PCM_Resistor_SMD_AKL:R_0603_1608Metric -> PCM_Resistor_SMD_AKL:R_0402_1005Metric
- R13: renamed from R22; footprint PCM_Resistor_SMD_AKL:R_0603_1608Metric -> PCM_Resistor_SMD_AKL:R_0402_1005Metric
- R14: renamed from R6; footprint PCM_Resistor_SMD_AKL:R_0603_1608Metric -> PCM_Resistor_SMD_AKL:R_0402_1005Metric
- R15: renamed from R9; footprint PCM_Resistor_SMD_AKL:R_0603_1608Metric -> PCM_Resistor_SMD_AKL:R_0402_1005Metric
- R16: renamed from R10; footprint PCM_Resistor_SMD_AKL:R_0603_1608Metric -> PCM_Resistor_SMD_AKL:R_0402_1005Metric
- R17: renamed from R21; footprint PCM_Resistor_SMD_AKL:R_0603_1608Metric -> PCM_Resistor_SMD_AKL:R_0402_1005Metric
- R18: renamed from R23; footprint PCM_Resistor_SMD_AKL:R_0603_1608Metric -> PCM_Resistor_SMD_AKL:R_0402_1005Metric
- R19: renamed from R24; footprint PCM_Resistor_SMD_AKL:R_0603_1608Metric -> PCM_Resistor_SMD_AKL:R_0402_1005Metric
- R2: renamed from R8; footprint PCM_Resistor_SMD_AKL:R_0603_1608Metric -> PCM_Resistor_SMD_AKL:R_0402_1005Metric
- R20: renamed from R25; footprint PCM_Resistor_SMD_AKL:R_0603_1608Metric -> PCM_Resistor_SMD_AKL:R_0402_1005Metric
- R21: renamed from R13; footprint PCM_Resistor_SMD_AKL:R_0603_1608Metric -> PCM_Resistor_SMD_AKL:R_0402_1005Metric
- R22: renamed from R14; footprint PCM_Resistor_SMD_AKL:R_0603_1608Metric -> PCM_Resistor_SMD_AKL:R_0402_1005Metric
- R23: renamed from R11; footprint PCM_Resistor_SMD_AKL:R_0603_1608Metric -> PCM_Resistor_SMD_AKL:R_0402_1005Metric
- R24: renamed from R12; footprint PCM_Resistor_SMD_AKL:R_0603_1608Metric -> PCM_Resistor_SMD_AKL:R_0402_1005Metric
- R25: renamed from R19; footprint PCM_Resistor_SMD_AKL:R_0603_1608Metric -> PCM_Resistor_SMD_AKL:R_0402_1005Metric
- R26: renamed from R20; footprint PCM_Resistor_SMD_AKL:R_0603_1608Metric -> PCM_Resistor_SMD_AKL:R_0402_1005Metric
- R3: renamed from R15; footprint PCM_Resistor_SMD_AKL:R_0603_1608Metric -> PCM_Resistor_SMD_AKL:R_0402_1005Metric
- R4: renamed from R16; footprint PCM_Resistor_SMD_AKL:R_0603_1608Metric -> PCM_Resistor_SMD_AKL:R_0402_1005Metric
- R5: renamed from R2; footprint PCM_Resistor_SMD_AKL:R_0603_1608Metric -> PCM_Resistor_SMD_AKL:R_0402_1005Metric
- R6: renamed from R1; footprint PCM_Resistor_SMD_AKL:R_0603_1608Metric -> PCM_Resistor_SMD_AKL:R_0402_1005Metric
- R7: renamed from R26; footprint PCM_Resistor_SMD_AKL:R_0603_1608Metric -> PCM_Resistor_SMD_AKL:R_0402_1005Metric
- R8: renamed from R5; footprint PCM_Resistor_SMD_AKL:R_0603_1608Metric -> PCM_Resistor_SMD_AKL:R_0402_1005Metric
- R9: renamed from R4; footprint PCM_Resistor_SMD_AKL:R_0603_1608Metric -> PCM_Resistor_SMD_AKL:R_0402_1005Metric
- SW3: renamed from SW1; value MST-12D18G5 -> JS102011SAQN
- moved R1 131.6 mm to (156.2, 65.0), turned to 90 degrees
- moved R17 126.1 mm to (156.8, 52.5)
- moved R18 119.8 mm to (156.8, 51.2)
- moved C1 116.1 mm to (157.5, 65.0), turned to -90 degrees
- moved R15 107.6 mm to (137.2, 69.5)
- moved C8 106.8 mm to (156.8, 69.0), turned to -90 degrees
- moved R2 106.3 mm to (135.0, 50.0), turned to -90 degrees
- moved R16 105.4 mm to (135.1, 72.0), turned to 90 degrees
- moved R11 102.1 mm to (135.2, 60.8), turned to -90 degrees
- moved R10 102.1 mm to (135.2, 58.5), turned to 90 degrees
- moved R26 100.5 mm to (131.2, 53.1), turned to 90 degrees
- moved R22 100.1 mm to (124.5, 48.5), turned to 90 degrees
- moved R25 99.1 mm to (130.8, 54.6), turned to 180 degrees
- moved R14 99.0 mm to (123.8, 65.2), turned to -90 degrees
- moved R24 98.4 mm to (125.5, 52.8), turned to 90 degrees
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- renumbered D7 to D11, D3 to D2, D11 to D3, D2 to D4, D4 to D5, D8 to D7, D9 to D8, D5 to D9, H3 to H2, H2 to H3, J2 to J1, J1 to J2, J4 to J3, J5 to J4, Q2 to Q1, Q1 to Q2, SW2 to SW1, SW3 to SW2, U5 to U1, U1 to U2, U6 to U3, U7 to U4, U2 to U5, U8 to U6, U3 to U7, U4 to U8
Connections:
- D7 pad 4: /SUB_URXD_C -> /SUB_UTXD_C
- D7 pad 6: /SUB_UTXD_C -> /SUB_URXD_C
- J1 pad SH: unconnected-(J2-SHIELD-PadSH)_2 -> Net-(J1-SHIELD)
- J3 pad 3: /SUB_UTXD_C -> /SUB_URXD_C
- J3 pad 4: /SUB_URXD_C -> /SUB_UTXD_C
- LS1 pad 1: Net-(U3-OUTP) -> Net-(U7-OUTN)
- LS1 pad 2: Net-(U3-OUTN) -> Net-(U7-OUTP)
- R10 pad 1: /SUB_I2C_SDA -> /SUB_I2C_SCL
- R11 pad 1: /SUB_I2C_SCL -> /SUB_I2C_SDA
- R17 pad 1: /SUB_UART_TXD -> /SUB_UART_RXD
- R18 pad 1: /SUB_UART_RXD -> /SUB_UART_TXD
- U2 pad 10: /SUB_I2C_SDA -> /SUB_I2C_SCL
- U2 pad 11: /SUB_I2C_SCL -> /SUB_I2C_SDA
- U2 pad 12: /I2S_IN_DATA -> /SUB_AUX1/ID0
- U2 pad 15: /BATT_V -> /VSUB_CTRL
- U2 pad 16: /RGB_CLK -> /SUB_EN
- U2 pad 17: /I2S_IN_WS -> /I2S_IN_DATA
- U2 pad 19: /I2S_OUT_DATA -> /I2S_IN_WS
- U2 pad 20: /I2S_OUT_BCLK -> /I2S_OUT_DATA
- U2 pad 21: /I2S_OUT_LRCLK -> /I2S_OUT_BCLK
- U2 pad 22: /IMU_SDA -> /I2S_OUT_LRCLK
- U2 pad 23: /VSUB_CTRL -> /RGB_DATA
- U2 pad 24: /RGB_DATA -> /RGB_CLK
- U2 pad 25: /SUB_EN -> /SUB_AUX2
- U2 pad 31: /LCD_DIN -> /LCD_RST
- U2 pad 32: /LCD_CLK -> /LCD_DC
- U2 pad 34: /LCD_DC -> /LCD_CLK
- U2 pad 35: /LCD_RST -> /LCD_DIN
- U2 pad 38: /SUB_V -> /SUB_AUX3
- U2 pad 5: /SUB_AUX1/ID0 -> /BATT_V
- U2 pad 6: /SUB_AUX2 -> /SUB_V
- U2 pad 7: /SUB_AUX3 -> /IMU_INT1
- U2 pad 8: /IMU_SCL -> /IMU_SDA
- U2 pad 9: /IMU_INT1 -> /IMU_SCL
- U7 pad 10: Net-(U3-OUTN) -> Net-(U7-OUTN)
- U7 pad 9: Net-(U3-OUTP) -> Net-(U7-OUTP)
Routing:
- net +VSW: track 0.00 -> 106.5 mm, vias 0 -> 8
- net Net-(D7-L2-Pad3): track 0.00 -> 52.7 mm, vias 0 -> 2
- net VBUS: track 0.00 -> 52.4 mm, vias 0 -> 4
- net Net-(D7-L1-Pad1): track 0.00 -> 51.4 mm, vias 0 -> 2
- net GND: track 0.00 -> 48.8 mm, vias 0 -> 59
- net /SUB_EN: track 0.00 -> 32.0 mm, vias 0 -> 1
- net VSUB: track 0.00 -> 28.8 mm, vias 0 -> 2
- net +VPW: track 0.00 -> 28.5 mm, vias 0 -> 3
- net /SUB_AUX3: track 0.00 -> 27.6 mm, vias 0 -> 1
- net Net-(D8-L1-Pad1): track 0.00 -> 25.2 mm, vias 0 -> 2
- net /SUB_AUX1/ID0: track 0.00 -> 24.3 mm, vias 0 -> 1
- net Net-(D8-L2-Pad3): track 0.00 -> 22.4 mm, vias 0 -> 2
- net Net-(J1-SHIELD): track 0.00 -> 20.5 mm
- net /ESP_USB_D-: track 0.00 -> 20.1 mm
- net /ESP_USB_D+: track 0.00 -> 20.0 mm
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- added copper zone on B.Cu, net +3V3
- added copper zone on In1.Cu, net GND
- added copper zone on In2.Cu, net GND
Other:
- board size 56.5 x 34 mm -> 58 x 35 mm

Commit message: added silkscreen and moved reset button to right side
Parts:
- added Ref**: Val**, PCM_SparkFun-Aesthetic:OSHW_Logo_5mm, F.Cu at (130.2, 46.0)
- moved SW2 28.5 mm to (158.8, 48.5)
Routing:
- net /ESP_EN: track 9.19 -> 28.1 mm, vias 0 -> 2
- net GND: track 48.8 -> 49.7 mm
Other:
- board text added: "20/07/26"
- board text added: "BOOT0"
- board text added: "EN"
- board text added: "ESP-HI-PLUS v1"
- board text added: "JLCJLCJLCJLC"
- board text added: "MAG1"
- board text added: "MAG2"

Commit message: Added Sub-module Configuration Resistor and Resistor Table
Parts:
- added R28: 47k, PCM_Resistor_SMD_AKL:R_0402_1005Metric, F.Cu at (131.0, 61.5)
- added R29: 47k, PCM_Resistor_SMD_AKL:R_0402_1005Metric, F.Cu at (133.0, 61.5)
- J2: value 0.71" LCD -> 2" IPS LCD
Routing:
- net /SUB_AUX1/ID0: track 24.3 -> 30.5 mm
- net +3V3: track 19.9 -> 21.0 mm
- net GND: track 49.7 -> 50.2 mm, vias 59 -> 60
