File: Sub-modules/Robot/Robot.kicad_pcb (KiCad board)
At the start: 2 copper layers, 70.1 x 100 mm, 80 parts, among them J1 USB_C_Receptacle_USB2.0_14P, J2 JST-XH, J3 XT60, J4 JST-XH, J5 PR5L5015-5P-C-H, J6 PR5L5015-5P-C-H, J7 Conn_01x10_MountingPin, J8 Conn_01x10_MountingPin, M1 MG996R, M2 MG996R, M3 MG996R, M4 MG996R, Q1 NTK3139P, SW1 SKRPACE010, SW2 SKRPACE010, U1 W25Q16JVSS, U10 AT24CS02-SSHM, U2 MAX40200AUK, U3 RP2040, U4 UBEC-5V, U5 MAX40200AUK, U6 MAX17049, U7 LSM6DSV16X, U8 TLV75733PDBV, U9 INA3221, Y1 ABM8-272-T3

Commit message: upgrade Robot submodule to 3S battery
Parts:
- added C18: 0u1, Capacitor_SMD:C_0402_1005Metric, F.Cu at (144.9, 62.0)
- added LED1: Broadcom_ASMB-KTF0-0A306, PCM_LED_SMD_AKL:LED_ASMB-KTF0-0A306, F.Cu at (151.4, 59.2)
- added R19: 150, PCM_Resistor_SMD_AKL:R_0402_1005Metric, F.Cu at (154.4, 58.5)
- added R20: 150, PCM_Resistor_SMD_AKL:R_0402_1005Metric, F.Cu at (148.7, 58.5)
- added R21: 150, PCM_Resistor_SMD_AKL:R_0402_1005Metric, F.Cu at (148.7, 60.0)
- added U11: NINA-B416, NINA-B416:NINA_LGA71R_1500X1000X223_PCB, F.Cu at (148.2, 67.8)
- moved C10 0.71 mm to (162.5, 94.8), turned to 90 degrees
Connections:
- U3 pad 4: unconnected-(U3-GPIO2-Pad4) -> /BLE_SW1
- U3 pad 5: unconnected-(U3-GPIO3-Pad5) -> /BLE_UART_RX
- U3 pad 6: unconnected-(U3-GPIO4-Pad6) -> /BLE_UART_TX
- U3 pad 7: unconnected-(U3-GPIO5-Pad7) -> /BLE_UART_CTS
- U3 pad 8: unconnected-(U3-GPIO6-Pad8) -> /BLE_UART_RTS
- U3 pad 9: unconnected-(U3-GPIO7-Pad9) -> /BLE_SW2
Routing:
- net /BLE_SW1: track 0.00 -> 51.2 mm, vias 0 -> 2
- net /BLE_SW2: track 0.00 -> 35.1 mm, vias 0 -> 2
- net /BLE_UART_RTS: track 0.00 -> 33.9 mm, vias 0 -> 2
- net /BLE_UART_CTS: track 0.00 -> 33.6 mm, vias 0 -> 2
- net /BLE_UART_TX: track 0.00 -> 33.2 mm, vias 0 -> 2
- net /BLE_UART_RX: track 0.00 -> 32.7 mm, vias 0 -> 2
- net /BLE_RED: track 0.00 -> 5.58 mm
- net /BLE_BLUE: track 0.00 -> 4.56 mm, vias 0 -> 2
- net +3V3: track 13.9 -> 17.1 mm, vias 4 -> 6
- net Net-(LED1-R): track 0.00 -> 1.65 mm
- net Net-(LED1-G): track 0.00 -> 1.39 mm
- net Net-(LED1-B): track 0.00 -> 1.39 mm
- net GND: track 56.7 -> 56.8 mm, vias 47 -> 66
