File: Sub-modules/Robot/Robot.kicad_sch (KiCad schematic)
At the start: 70 parts, among them J1 USB_C_Receptacle_USB2.0_14P, J2 PR5L5015-5P-C-H, J3 PR5L5015-5P-C-H, J4 XT60, J5 JST-XH, J6 JST-XH, M1 MG996R, M2 MG996R, M3 MG996R, M4 MG996R, Q2 NTK3139P, SW1 SKRPACE010, SW3 SKRPACE010, U1 W25Q16JVSS, U10 AT24CS02-SSHM, U11 INA3221, U2 MAX40200AUK, U3 RP2040, U4 TLV75733PDBV, U5 MAX17049, U6 MAX40200AUK, U7 UBEC-5V, U8 LSM6DSV16X, Y1 ABM8-272-T3

Commit message: Robot v1.0
Parts:
- added H1, H2, H3, H4, H5, H6: MountingHole_Pad_MP, MountIngHole_M3_Slim:MountingHole_M3_Slim, symbol Mechanical:MountingHole_Pad_MP
- added J7, J8: Conn_01x10_MountingPin, Connector_FFC-FPC:Hirose_FH12-10S-0.5SH_1x10-1MP_P0.50mm_Horizontal, symbol Connector_Generic_MountingPin:Conn_01x10_MountingPin
- BT1: renamed from BT2; footprint (none) -> Connector_AMASS:AMASS_XT60-F_1x02_P7.20mm_Vertical
- R11: renamed from R13; value 383k -> 953k
- R8: renamed from R14; footprint (none) -> PCM_Resistor_SMD_AKL:R_1206_3216Metric; symbol PCM_Resistor_AKL:R_Shunt_Generic -> Device:R_Small
- R9: renamed from R1; footprint (none) -> PCM_Resistor_SMD_AKL:R_1206_3216Metric; symbol PCM_Resistor_AKL:R_Shunt_Generic -> Device:R_Small
- U4: renamed from U7; footprint (none) -> UBEC-5V:UBEC-5V
- renumbered C3 to C1, C20 to C10, C21 to C11, C23 to C12, C15 to C13, C8 to C14, C10 to C15, C22 to C16, C18 to C17, C1 to C2, C2 to C3, C5 to C4, C11 to C5, C9 to C6, C19 to C7, C6 to C8, C7 to C9, D6 to D1, D1 to D2, J5 to J2, J4 to J3, J6 to J4, J2 to J5, J3 to J6, Q2 to Q1, R3 to R1, R15 to R10, R9 to R12, R10 to R13, R11 to R14, R12 to R15, R4 to R3, R5 to R4, R6 to R5, R7 to R6, R8 to R7, SW3 to SW2, U6 to U5, U5 to U6, U8 to U7, U4 to U8, U11 to U9
Connections:
- net GND: now also H1.MP, H2.MP, H3.MP, H4.MP, H5.MP, H6.MP, J7.2 (Pin_2), J8.9 (Pin_9)
- net IMU_INT1: now also U3.13 (GPIO10); no longer U3.16 (GPIO13)
- net PWM0: now also U3.30 (GPIO19); no longer U3.6 (GPIO4)
- net PWM1: now also U3.32 (GPIO21); no longer U3.7 (GPIO5)
- net PWM2: now also U3.35 (GPIO23); no longer U3.8 (GPIO6)
- net PWM3: now also U3.37 (GPIO25); no longer U3.9 (GPIO7)
- net PWR_CRIT: now also U3.34 (GPIO22); no longer U3.18 (GPIO15)
- net PWR_PV: now also U3.31 (GPIO20); no longer U3.17 (GPIO14)
- net PWR_TC: no longer U3.28 (GPIO17)
- net PWR_WARN: now also U3.36 (GPIO24); no longer U3.27 (GPIO16)
- net PWR_~{ALERT}: now also U3.12 (GPIO9)
- net RGB_CLK: now also U3.18 (GPIO15)
- net RGB_DATA: now also U3.11 (GPIO8)
- net SUB_AUX1/ID0: now also U3.27 (GPIO16), J7.8 (Pin_8), J8.3 (Pin_3)
- net SUB_AUX2: now also U3.28 (GPIO17), J7.9 (Pin_9), J8.2 (Pin_2)
- net SUB_AUX3: now also U3.29 (GPIO18), J7.10 (Pin_10), J8.1 (Pin_1)
- net SUB_EN: now also J7.5 (Pin_5), J8.6 (Pin_6)
- net SUB_I2C_SCL: now also R14.1; no longer R15.1
- net SUB_I2C_SDA: now also R15.1; no longer R14.1
- net SUB_ISCL_C: now also D5.6 (L1); no longer D5.4 (L2)
- net SUB_ISDA_C: now also D5.4 (L2); no longer D5.6 (L1)
- net SUB_UART_RXD: now also R12.1, U3.17 (GPIO14), J7.7 (Pin_7), J8.4 (Pin_4); no longer R13.1, U3.5 (GPIO3)
- net SUB_UART_TXD: now also R13.1, U3.16 (GPIO13), J7.6 (Pin_6), J8.5 (Pin_5); no longer R12.1, U3.4 (GPIO2)
- net SUB_URXD_C: now also D4.6 (L1); no longer D4.4 (L2)
- net SUB_UTXD_C: now also D4.4 (L2); no longer D4.6 (L1)
- net VBATT: now also F1.1, J3.1 (Pin_1); no longer F1.2, U4.1 (VIN+)
- net VBATT_MON: now also Q1.2 (S), R8.1, U4.3 (VOUT), U9.15 (IN+2); no longer R8.2, U9.12 (IN+1)
- net VBUS: no longer D3.1 (K)
- net VBUS_MON: now also Q1.3 (D), R9.1, U5.5 (OUT), U9.12 (IN+1); no longer R9.2, U9.15 (IN+2)
- net VSER: now also F2.1, F3.1, F4.1, F5.1, R8.2, U9.14 (IN-2); no longer R8.4
- net VSYS: now also D3.1 (K), R9.2, U9.11 (IN-1), J7.1 (Pin_1), J8.10 (Pin_10); no longer F2.1, F3.1, F4.1, F5.1, R9.4
- removed net VSER_MON: R8.3, U9.11 (IN-1)
- removed net VSYS_MON: R9.3, U9.14 (IN-2)
- new net: F1.2, U4.1 (VIN+), U4.5 (EN)
- no-connect marks 11 -> 17
Other:
- note added: "2-Terminal Shunt Resistors (for availability)"
- note added: "Sub-module Class 1: Actuator - Servo R_ID = 953k"
- note removed: "Sub-module Class 3: Sensor - Environmental R_ID = 383k"
- title: (none) -> Robot
- moved on the sheet: C13, C15, R6, R7, U7

Commit message: upgrade Robot submodule to 3S battery
Parts:
- removed U6: MAX17049, PCM_SparkFun-Semiconductor-Standard:DFN-8_2x2mm_P0.5mm_EP1.2x0.8mm, symbol PCM_SparkFun-IC-Power:MAX17048
- added C18: 0u1, Capacitor_SMD:C_0402_1005Metric, symbol Device:C_Small
- added C19: 470u, symbol Device:C_Polarized_Small
- added C20, C21: 470n, Capacitor_SMD:C_0402_1005Metric, symbol Device:C_Small
- added LED1: Broadcom_ASMB-KTF0-0A306, PCM_LED_SMD_AKL:LED_ASMB-KTF0-0A306, symbol PCM_LED_AKL:Broadcom_ASMB-KTF0-0A306
- added R19, R20, R21: 150, PCM_Resistor_SMD_AKL:R_0402_1005Metric, symbol Device:R_Small
- added R22: 50, PCM_Resistor_SMD_AKL:R_0402_1005Metric, symbol Device:R_Small
- added R23: 10m, PCM_Resistor_SMD_AKL:R_1206_3216Metric, symbol Device:R_Small
- added R24, R25: 10k, PCM_Resistor_SMD_AKL:R_0402_1005Metric, symbol Device:R_Small
- added TH1, TH2: 10k, symbol Device:Thermistor_NTC
- added U11: NINA-B416, NINA-B416:NINA_LGA71R_1500X1000X223_PCB, symbol NINA-B416:NINA-B416
- added U12: MAX17205, Package_DFN_QFN:TDFN-14-1EP_3x3mm_P0.4mm_EP1.78x2.35mm, symbol Robot Library:MAX17205
- BT1: value 2S/10C ~1500mAh -> 3S/10C ~1500mAh
- J2: footprint Connector_JST:JST_XH_S3B-XH-A_1x03_P2.50mm_Horizontal -> Connector_JST:JST_XH_S4B-XH-A_1x04_P2.50mm_Horizontal; symbol Connector_Generic:Conn_01x03 -> Connector_Generic:Conn_01x04
- J4: footprint Connector_JST:JST_XH_B3B-XH-A_1x03_P2.50mm_Vertical -> Connector_JST:JST_XH_B4B-XH-AM_1x04_P2.50mm_Vertical; symbol Connector_Generic:Conn_01x03 -> Connector_Generic:Conn_01x04
Connections:
- net +3V3: now also C18.1, LED1.1 (A), U11.10 (VCC), U11.31 (VBUS), U11.9 (VCC_IO)
- net PWR_~{ALERT}: now also U12.8 (ALRT1)
- net RP_I2C_SCL: now also U12.12 (SDA)
- net RP_I2C_SDA: now also U12.11 (SCL)
- net VBATT: now also R22.1
- net BLE_SW1: now reaches U3.4 (GPIO2)
- net BLE_SW1: now also R20.2, U11.7 (GREEN/SWITCH_1)
- net BLE_UART_RX: now reaches U3.5 (GPIO3)
- net BLE_UART_RX: now also U11.23 (UART_RXD)
- net BLE_UART_TX: now reaches U3.6 (GPIO4)
- net BLE_UART_TX: now also U11.22 (UART_TXD)
- net BLE_UART_CTS: now reaches U3.7 (GPIO5)
- net BLE_UART_CTS: now also U11.21 (UART_CTS)
- net BLE_UART_RTS: now reaches U3.8 (GPIO6)
- net BLE_UART_RTS: now also U11.20 (UART_RTS)
- net BLE_SW2: now reaches U3.9 (GPIO7)
- net BLE_SW2: now also U11.18 (SWITCH_2)
- net CELL2- renamed COM2
- net COM renamed COM1
- net GND renamed EGP57
- net EGP57: now also C18.2, C20.2, C21.2, R23.2, TH1.2, TH2.2, U11.12 (GND12), U11.14 (GND14), U11.26 (GND26), U11.30 (GND30), U11.53 (GND53), U11.56 (EGP56), U11.57 (EGP57), U11.58 (EGP58), U11.59 (EGP59), U11.6 (GND6), U11.60 (EGP60), U11.61 (EGP61), U11.62 (EGP62), U11.63 (EGP63), U11.64 (EGP64), U11.65 (EGP65), U11.66 (EGP66), U11.67 (EGP67), U12.13 (CELLX), U12.15 (EP), U12.4 (CSN), U12.6 (CELL2), U12.7 (CELL1); no longer BT1.2 (-)
- new net: R25.1, TH1.1, U12.9 (AIN1)
- new net: LED1.2 (R), R19.1
- new net: LED1.4 (B), R21.1
- new net: R24.1, TH2.1, U12.10 (AIN2)
- new net: R24.2, R25.2, U12.14 (THRM)
- new net: BT1.2 (-), R23.1, U12.2 (CSP)
- new net: R22.2, U12.5 (VBATT)
- new net: LED1.3 (G), R20.1
- new net: C21.1, U12.1 (REG3)
- new net: C20.1, U12.3 (REG2)
- new net BLE_BLUE: R21.2, U11.8 (BLUE)
- new net BLE_RED: R19.2, U11.1 (RED)
- new net CELL3-: J2.4 (Pin_4), J4.4 (Pin_4)
Other:
- moved on the sheet: BT1
