File: Sub-modules/Desktop/Desktop.kicad_pcb (KiCad board)
At the start: 2 copper layers, 60 x 43 mm, 56 parts, among them J1 USB_C_Receptacle_USB2.0_14P, J2 PR5L5015-5P-C-H, J3 PR5L5015-5P-C-H, SW1 SKRPACE010, SW2 SW_Push, SW3 SKRPACE010, U1 W25Q16JVSS, U10 AT24CS02-SSHM, U2 MAX40200AUK, U3 RP2040, U4 TLV75733PDBV, U5 SCD40-D-R2, U6 STHS34PF80, U7 VEML7700-TT, U8 MCP79410, Y1 ABM8-272-T3, Y2 X1A0000610006

Commit message: Desktop v1.15: revert to SHT40 for cost reduction
Parts:
- C16: moved to F.Cu
- U5: value SCD40-D-R2 -> SHT4x; footprint Sensor:Sensirion_SCD4x-1EP_10.1x10.1mm_P1.25mm_EP4.8x4.8mm -> Sensor_Humidity:Sensirion_DFN-4_1.5x1.5mm_P0.8mm_SHT4x_NoCentralPad
- moved U5 0.76 mm to (132.6, 48.2), turned to 90 degrees
Connections:
- U5 pad 1: (no net) -> /RP_I2C_SDA
- U5 pad 2: (no net) -> /RP_I2C_SCL
- U5 pad 3: (no net) -> +3V3
- U5 pad 4: (no net) -> GND
Routing:
- net GND: track 54.6 -> 51.2 mm, vias 51 -> 48
- net +3V3: track 188.7 -> 186.8 mm, vias 12 -> 11
- net /RP_I2C_SCL: track 59.7 -> 58.3 mm
- net /RP_I2C_SDA: track 56.4 -> 55.8 mm

Commit message: added new Keyboard submodule
Parts:
- added C17: 0u1, Capacitor_SMD:C_0402_1005Metric, F.Cu at (0.94, 0.48)
Changed lines of the file:
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@@
+		)
+	)
+	(footprint "Capacitor_SMD:C_0402_1005Metric"
+		(layer "F.Cu")
+		(at 0.935 0.485)
+		(descr "Capacitor SMD 0402 (1005 Metric), square (rectangular) end terminal, IPC-7351 nominal, (Body size source: IPC-SM-782 page 76, https://www.pcb-3d.com/wordpress/wp-content/uploads/ipc-sm-782a_amendment_1_and_2.pdf)")
+		(tags "capacitor")
+		(property "Reference" "C17"
+			(at 0 -1.16 0)
+			(layer "F.SilkS")
+			(effects
+				(font
+					(size 1 1)
+					(thickness 0.15)
+				)
+			)
+		)
+		(property "Value" "0u1"
+			(at 0 1.16 0)
+			(layer "F.Fab")
+			(effects
+				(font
+					(size 1 1)
+					(thickness 0.15)
+				)
+			)
+		)
+		(property "Datasheet" ""
+			(at 0 0 0)
+			(layer "F.Fab")
+			(hide yes)
+			(effects
+				(font
+					(size 1.27 1.27)
+				)
+			)
+		)
+		(property "Description" ""
+			(at 0 0 0)
+			(layer "F.Fab")
+			(hide yes)
+			(effects
+				(font
+					(size 1.27 1.27)
+				)
+			)
+		)
+		(property "KiLib_Generator" "SMD_2terminal_chip_molded"
+			(at 0 0 0)
+			(layer "F.SilkS")
+			(hide yes)
+			(effects
+				(font
+					(size 1 1)
+					(thickness 0.15)
+				)
+			)
+		)
+		(property ki_fp_filters "C_*")
+		(sheetname "/")
+		(sheetfile "Desktop.kicad_sch")
+		(units
+			(unit
+				(name "A")
+				(pins "1" "2")
+			)
+		)
+		(attr smd)
+		(duplicate_pad_numbers_are_jumpers no)
+		(fp_line
+			(start -0.107836 -0.36)
+			(end 0.107836 -0.36)
+			(stroke
+				(width 0.12)
+				(type solid)
+			)
+			(layer "F.SilkS")
+		)
+		(fp_line
+			(start -0.107836 0.36)
+			(end 0.107836 0.36)
+			(stroke
+				(width 0.12)
+				(type solid)
+			)
+			(layer "F.SilkS")
+		)
+		(fp_rect
+			(start -0.91 -0.46)
+			(end 0.91 0.46)
+			(stroke
+				(width 0.05)
+				(type solid)
+			)
+			(fill no)
+			(layer "F.CrtYd")
+		)
+		(fp_rect
+			(start -0.5 -0.25)
+			(end 0.5 0.25)
+			(stroke
+				(width 0.1)
+				(type solid)
+			)
+			(fill no)
+			(layer "F.Fab")
+		)
+		(fp_text user "${REFERENCE}"
+			(at 0 0 0)
+			(layer "F.Fab")
+			(effects
+				(font
+					(size 0.25 0.25)
+					(thickness 0.04)
+				)
+			)
+		)
+		(pad "1" smd roundrect
+			(at -0.48 0)
+			(size 0.56 0.62)
+			(layers "F.Cu" "F.Mask" "F.Paste")
+			(roundrect_rratio 0.25)
+			(net "GND")
+			(pintype "passive")
+		)
+		(pad "2" smd roundrect
+			(at 0.48 0)
+			(size 0.56 0.62)
+			(layers "F.Cu" "F.Mask" "F.Paste")
+			(roundrect_rratio 0.25)
+			(net "+3V3")
+			(pintype "passive")
+		)
+		(embedded_fonts no)
+		(model "${KICAD10_3DMODEL_DIR}/Capacitor_SMD.3dshapes/C_0402_1005Metric.step"
+			(offset
+				(xyz 0 0 0)
+			)
+			(scale
+				(xyz 1 1 1)
+			)
+			(rotate
+				(xyz 0 0 0)
+			)
 		)
 	)

Commit message: Desktop v1.15: Changed I2C pins to 10 and 11 to fix I2C incompatibility issue, changed RGB LED to Neopixel
Parts:
- added D6: RED, LED_SMD:LED_0805_2012Metric, F.Cu at (156.5, 79.0)
- added D7: GREEN, LED_SMD:LED_0805_2012Metric, F.Cu at (140.5, 76.0)
- added JP1: SolderJumper_3_Bridged12, Jumper:SolderJumper-3_P1.3mm_Bridged12_RoundedPad1.0x1.5mm, F.Cu at (152.0, 78.5)
- added R14: 5k1, PCM_Resistor_SMD_AKL:R_0402_1005Metric, F.Cu at (156.5, 82.0)
- added R15: 5k1, PCM_Resistor_SMD_AKL:R_0402_1005Metric, F.Cu at (141.5, 70.0)
- D2: value SK9822-EC20 -> WS2812B-2020; footprint PCM_SparkFun-LED:APA102_2020-6Pin -> LED_SMD:LED_WS2812B-2020_PLCC4_2.0x2.0mm
- moved C17 157.3 mm to (140.5, 73.0), turned to 90 degrees
- moved U6 17.8 mm to (139.5, 47.0)
- moved C16 17.7 mm to (137.0, 47.5)
- moved D2 0.78 mm to (142.5, 73.0), turned to 90 degrees
Connections:
- D2 pad 4: /RGB_CLK -> +3V3
- U3 pad 13: unconnected-(U3-GPIO10-Pad13) -> /RP_I2C_SDA
- U3 pad 14: /RP_I2C_SDA -> /RP_I2C_SCL
- U3 pad 15: /RP_I2C_SCL -> unconnected-(U3-GPIO12-Pad15)
- U3 pad 36: /RGB_CLK -> /LED_PIN
- U4 pad 3: /SUB_EN -> Net-(JP1-A)
Routing:
- net /PS_INT: track 53.2 -> 35.7 mm
- net /RP_I2C_SCL: track 58.3 -> 65.0 mm
- net Net-(D7-K): track 0.00 -> 6.25 mm, vias 0 -> 2
- net /RGB_CLK: track 5.91 -> 0.00 mm
- net /SUB_EN: track 8.76 -> 3.46 mm
- net /RP_I2C_SDA: track 55.8 -> 60.2 mm, vias 6 -> 7
- net VBUS: track 52.9 -> 56.1 mm
- net Net-(JP1-A): track 0.00 -> 2.70 mm
- net +3V3: track 186.8 -> 188.9 mm
- net /LED_PIN: track 0.00 -> 1.70 mm
- net GND: track 51.2 -> 52.8 mm, vias 48 -> 50
- net Net-(D6-K): track 0.00 -> 1.55 mm
- net /QSPI_SD1: track 20.9 -> 21.9 mm
Other:
- board text added: "IND"
- board text added: "SUB"
