File: Sub-modules/Keyboard/Keyboard.kicad_sch (KiCad schematic)
At the start: 42 parts, among them J1 USB_C_Receptacle_USB2.0_14P, J2 PR5L5015-5P-C-H, J3 PR5L5015-5P-C-H, SW1 SKRPACE010, SW3 SKRPACE010, SW4 SW_Push_45deg, U1 W25Q16JVSS, U10 AT24CS02-SSHM, U2 MAX40200AUK, U3 RP2040, U4 TLV75733PDBV, Y1 ABM8-272-T3

Commit message: assign footprints to keyswitch and diodes
Parts:
- D2: footprint (none) -> Diode_SMD:D_SOD-123
- SW4: footprint (none) -> PCM_Switch_Keyboard_Hotswap_Kailh:SW_Hotswap_Kailh_MX_1.00u
Changed lines of the file:
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@@
 			)
 		)
-		(property "Footprint" ""
+		(property "Footprint" "Diode_SMD:D_SOD-123"
 			(at 139.7 154.94 90)
 			(hide yes)
@@
 			)
 		)
-		(property "Footprint" ""
+		(property "Footprint" "PCM_Switch_Keyboard_Hotswap_Kailh:SW_Hotswap_Kailh_MX_1.00u"
 			(at 137.16 149.86 0)
 			(hide yes)

Commit message: updated Keyboard
Parts:
- removed C1, C21, C5: 1u, Capacitor_SMD:C_0402_1005Metric, symbol Device:C_Small
- removed C19, C2, C20, C9: 0u1, Capacitor_SMD:C_0402_1005Metric, symbol Device:C_Small
- removed C3: 4n7, Capacitor_SMD:C_0402_1005Metric, symbol Device:C_Small
- removed C6, C7: 15p, Capacitor_SMD:C_0402_1005Metric, symbol Device:C_Small
- removed D1: USBLC6-2P6, PCM_Package_TO_SOT_SMD_AKL:SOT-666, symbol PCM_Diode_TVS_AKL:USBLC6-2P6
- removed D2: D_Schottky_Small, Diode_SMD:D_SOD-123, symbol Device:D_Schottky_Small
- removed D6: SK9822-EC20, PCM_SparkFun-LED:APA102_2020-6Pin, symbol PCM_SparkFun-LED:APA102_2020-6Pin
- removed J1: USB_C_Receptacle_USB2.0_14P, Connector_USB:USB_C_Receptacle_HCTL_HC-TYPE-C-16P-01A, symbol Connector:USB_C_Receptacle_USB2.0_14P
- removed R2, R6: 1k, PCM_Resistor_SMD_AKL:R_0402_1005Metric, symbol Device:R_Small
- removed R3: 1M, PCM_Resistor_SMD_AKL:R_0402_1005Metric, symbol Device:R_Small
- removed R4, R5: 5k1, PCM_Resistor_SMD_AKL:R_0402_1005Metric, symbol Device:R_Small
- removed SW1, SW3: SKRPACE010, Button_Switch_SMD:SW_Push_1P1T_NO_Vertical_Wuerth_434133025816, symbol Switch:SW_Push
- removed U1: W25Q16JVSS, Package_SO:SOIC-8_5.3x5.3mm_P1.27mm, symbol Memory_Flash:W25Q16JVSS
- removed U2: MAX40200AUK, Package_TO_SOT_SMD:SOT-23-5, symbol Analog_Switch:MAX40200AUK
- removed U3: RP2040, Package_DFN_QFN:QFN-56-1EP_7x7mm_P0.4mm_EP3.2x3.2mm, symbol MCU_RaspberryPi:RP2040
- removed Y1: ABM8-272-T3, PCM_Crystal_AKL:Crystal_SMD_3225-4Pin_3.2x2.5mm, symbol Device:Crystal_GND24_Small
- added D10, D11, D12, D13, D14, D15, D16, D17, D18, D19, D20, D21, D22, D23, D24, D25, D26, D27, D28, D29, D30, D31, D32, D33, D34, D35, D36, D37, D38, D39, D40, D41, D42, D43, D44, D45, D46, D47, D48, D49, D50, D51, D52, D53, D54, D55, D56, D57, D58, D59, D60, D8, D9: BAT54-02V, PCM_Diode_SMD_AKL:D_SOD-523, symbol PCM_Diode_Schottky_AKL:BAT54-02V
- added D7: WS2812B-2020, LED_SMD:LED_WS2812B-2020_PLCC4_2.0x2.0mm, symbol LED:WS2812B-2020
- added SW10, SW11, SW12, SW13, SW14, SW15, SW16, SW17, SW18, SW19, SW20, SW21, SW22, SW23, SW24, SW25, SW26, SW27, SW28, SW29, SW30, SW31, SW32, SW33, SW34, SW35, SW36, SW37, SW38, SW39, SW40, SW41, SW42, SW43, SW44, SW45, SW46, SW47, SW48, SW49, SW5, SW50, SW51, SW6, SW7, SW8, SW9: SW_Push_45deg, Switch_Keyboard_Hotswap_Kailh:SW_Hotswap_Kailh_Choc_V1V2_1.00u, symbol Switch:SW_Push_45deg
- added SW52, SW53, SW55, SW56: SW_Push_45deg, Switch_Keyboard_Hotswap_Kailh:SW_Hotswap_Kailh_Choc_V1V2_1.25u, symbol Switch:SW_Push_45deg
- added SW54: SW_Push_45deg, Switch_Keyboard_Hotswap_Kailh:SW_Hotswap_Kailh_Choc_V1V2_2.00u, symbol Switch:SW_Push_45deg
- added U5: RP2040 ProMicro, pro_micro_rp2040:pro_micro_rp2040, symbol pro_micro_rp2040:pro_micro_rp2040
- SW4: footprint PCM_Switch_Keyboard_Hotswap_Kailh:SW_Hotswap_Kailh_MX_1.00u -> Switch_Keyboard_Hotswap_Kailh:SW_Hotswap_Kailh_Choc_V1V2_1.00u
Connections:
- net +3V3: now also D7.4 (VDD)
- net GND: now also D7.2 (VSS)
- net at SW4.2: now also D8.2 (A)
- net C1: now reaches SW4.1
- net C1: now also SW10.1, SW16.1, SW22.1
- new net: D49.2 (A), SW45.2
- new net: D28.2 (A), SW24.2
- new net: D42.2 (A), SW38.2
- new net: D30.2 (A), SW26.2
- new net: D40.2 (A), SW36.2
- new net: D39.2 (A), SW35.2
- new net: D13.2 (A), SW9.2
- new net: D27.2 (A), SW23.2
- new net: D52.2 (A), SW48.2
- new net: D37.2 (A), SW33.2
- new net: D44.2 (A), SW40.2
- new net: D34.2 (A), SW30.2
- new net: D38.2 (A), SW34.2
- new net: D33.2 (A), SW29.2
- new net: D57.2 (A), SW53.2
- new net: D9.2 (A), SW5.2
- new net: D20.2 (A), SW16.2
- new net: D41.2 (A), SW37.2
- new net: D35.2 (A), SW31.2
- new net: D12.2 (A), SW8.2
- new net: D46.2 (A), SW42.2
- new net: D56.2 (A), SW52.2
- new net: D24.2 (A), SW20.2
- new net: D55.2 (A), SW51.2
- new net: D59.2 (A), SW55.2
- new net: D50.2 (A), SW46.2
- new net: D36.2 (A), SW32.2
- new net: D43.2 (A), SW39.2
- new net: D48.2 (A), SW44.2
- new net: D25.2 (A), SW21.2
- new net: D14.2 (A), SW10.2
- new net: D45.2 (A), SW41.2
- new net: D19.2 (A), SW15.2
- new net: D51.2 (A), SW47.2
- new net: D22.2 (A), SW18.2
- new net: D47.2 (A), SW43.2
- new net: D21.2 (A), SW17.2
- new net: D18.2 (A), SW14.2
- new net: D53.2 (A), SW49.2
- new net: D17.2 (A), SW13.2
- new net: D32.2 (A), SW28.2
- new net: D11.2 (A), SW7.2
- new net: D23.2 (A), SW19.2
- new net: D10.2 (A), SW6.2
- new net: D26.2 (A), SW22.2
- new net: D16.2 (A), SW12.2
- new net: D60.2 (A), SW56.2
- new net: D29.2 (A), SW25.2
- new net: D15.2 (A), SW11.2
- new net: D58.2 (A), SW54.2
- new net: D31.2 (A), SW27.2
- new net: D54.2 (A), SW50.2
- new net BL_RGB: U5.24 (GP24)
- new net C10: SW40.1, SW41.1, SW42.1, SW43.1
- new net C11: SW44.1, SW45.1, SW46.1, SW47.1
- new net C12: SW48.1, SW49.1, SW50.1, SW51.1
- new net C13: SW54.1, U5.13 (GP13)
- new net C2: SW11.1, SW17.1, SW23.1, SW5.1
- new net C3: SW12.1, SW18.1, SW24.1, SW6.1
- new net C4: SW13.1, SW19.1, SW25.1, SW7.1
- new net C5: SW14.1, SW20.1, SW26.1, SW52.1, SW8.1
- new net C6: SW15.1, SW21.1, SW27.1, SW53.1, SW9.1
- new net C7: SW28.1, SW29.1, SW30.1, SW31.1, SW55.1
- new net C8: SW32.1, SW33.1, SW34.1, SW35.1, SW56.1
- new net C9: SW36.1, SW37.1, SW38.1, SW39.1
- new net R1: D10.1 (K), D11.1 (K), D12.1 (K), D13.1 (K), D8.1 (K), D9.1 (K)
- new net R2: D14.1 (K), D15.1 (K), D16.1 (K), D17.1 (K), D18.1 (K), D19.1 (K)
- new net R3: D20.1 (K), D21.1 (K), D22.1 (K), D23.1 (K), D24.1 (K), D25.1 (K)
- new net R4: D26.1 (K), D27.1 (K), D28.1 (K), D29.1 (K), D30.1 (K), D31.1 (K), U5.12 (GP12)
- new net R5: D32.1 (K), D36.1 (K), D40.1 (K), D44.1 (K), D48.1 (K), D52.1 (K)
- new net R6: D33.1 (K), D37.1 (K), D41.1 (K), D45.1 (K), D49.1 (K), D53.1 (K)
- new net R7: D34.1 (K), D38.1 (K), D42.1 (K), D46.1 (K), D50.1 (K), D54.1 (K), U5.16 (GP16)
- new net R8: D35.1 (K), D39.1 (K), D43.1 (K), D47.1 (K), D51.1 (K), D55.1 (K), U5.15 (GP15)
- new net R9: D56.1 (K), D57.1 (K), D58.1 (K), D59.1 (K), D60.1 (K), U5.14 (GP14)
- new net STAT_RGB: D7.3 (DIN), U5.11 (GP11)
- no-connect marks 6 -> 3
Other:
- note removed: "BOOTSEL"
- moved on the sheet: C17, SW4
